File: KiCad/battery.kicad_sch (KiCad schematic)
At the start: 7 parts, among them J2 Conn_01x02_Socket, U12 BQ25185DLHR

Commit message: Mods
Parts:
- removed BT1: BC-2013, JetBoard:BAT_BC-2013, symbol Connector:BC-2013
- U12: symbol 2025-03-10_01-20-10:BQ25185DLHR -> JetBoard:BQ25185DLHR
Connections:
- net CHARGE_EN# renamed ~{CHARGE_EN}
Changed lines of the file:
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@@
-	)
-	(junction
-		(at 210.82 99.06)
-		(diameter 0)
-		(color 0 0 0 0)
 	)
 	(junction
@@
 		(color 0 0 0 0)
 	)
-	(junction
-		(at 180.34 119.38)
-		(diameter 0)
-		(color 0 0 0 0)
-	)
 	(no_connect
 		(at 116.84 101.6)
@@
 	(wire
 		(pts
-			(xy 180.34 119.38) (xy 180.34 121.92)
+			(xy 180.34 109.22) (xy 180.34 121.92)
 		)
 		(stroke
@@
 	(wire
 		(pts
-			(xy 180.34 109.22) (xy 180.34 119.38)
-		)
-		(stroke
-			(width 0)
-			(type default)
-		)
-	)
-	(wire
-		(pts
-			(xy 210.82 99.06) (xy 210.82 101.6)
-		)
-		(stroke
-			(width 0)
-			(type default)
-		)
-	)
-	(wire
-		(pts
 			(xy 157.48 106.68) (xy 157.48 111.76)
 		)
@@
 	(wire
 		(pts
-			(xy 210.82 119.38) (xy 210.82 116.84)
-		)
-		(stroke
-			(width 0)
-			(type default)
-		)
-	)
-	(wire
-		(pts
 			(xy 157.48 119.38) (xy 157.48 121.92)
 		)
@@
 		(pts
 			(xy 165.1 101.6) (xy 165.1 106.68)
-		)
-		(stroke
-			(width 0)
-			(type default)
-		)
-	)
-	(wire
-		(pts
-			(xy 180.34 119.38) (xy 210.82 119.38)
 		)
 		(stroke
@@
 		)
 	)
-	(hierarchical_label "CHARGE_EN#"
+	(hierarchical_label "~{CHARGE_EN}"
 		(shape input)
 		(at 93.98 93.98 180)
@@
 	)
 	(symbol
-		(lib_id "2025-03-10_01-20-10:BQ25185DLHR")
+		(lib_id "JetBoard:BQ25185DLHR")
 		(at 135.89 96.52 0)
 		(unit 1)
@@
 		(fields_autoplaced yes)
 		(property "Reference" "U12"
-			(at 132.588 78.74 0)
+			(at 137.16 78.74 0)
 			(effects
 				(font
@@
 		)
 		(property "Value" "BQ25185DLHR"
-			(at 131.826 80.772 0)
+			(at 137.16 81.28 0)
 			(effects
 				(font
@@
 					(unit 1)
 				)
-			)
-		)
-	)
-	(symbol
-		(lib_id "Connector:BC-2013")
-		(at 210.82 109.22 270)
-		(unit 1)
-		(exclude_from_sim no)
-		(in_bom yes)
-		(on_board yes)
-		(dnp no)
-		(fields_autoplaced yes)
-		(property "Reference" "BT1"
-			(at 214.63 107.8229 90)
-			(effects
-				(font
-					(size 1.27 1.27)
-				)
-				(justify left)
-			)
-		)
-		(property "Value" "BC-2013"
-			(at 214.63 110.3629 90)
-			(effects
-				(font
-					(size 1.27 1.27)
-				)
-				(justify left)
-			)
-		)
-		(property "Footprint" "JetBoard:BAT_BC-2013"
-			(at 210.82 109.22 0)
-			(effects
-				(font
-					(size 1.27 1.27)
-				)
-				(justify bottom)
-				(hide yes)
-			)
-		)
-		(property "Datasheet" ""
-			(at 210.82 109.22 0)
-			(effects
-				(font
-					(size 1.27 1.27)
-				)
-				(hide yes)
-			)
-		)
-		(property "Description" ""
-			(at 210.82 109.22 0)
-			(effects
-				(font
-					(size 1.27 1.27)
-				)
-				(hide yes)
-			)
-		)
-		(property "PARTREV" "D"
-			(at 210.82 109.22 0)
-			(effects
-				(font
-					(size 1.27 1.27)
-				)
-				(justify bottom)
-				(hide yes)
-			)
-		)
-		(property "STANDARD" "Manufacturer Recommendations"
-			(at 210.82 109.22 0)
-			(effects
-				(font
-					(size 1.27 1.27)
-				)
-				(justify bottom)
-				(hide yes)
-			)
-		)
-		(property "MAXIMUM_PACKAGE_HEIGHT" "3.68mm"
-			(at 210.82 109.22 0)
-			(effects
-				(font
-					(size 1.27 1.27)
-				)
-				(justify bottom)
-				(hide yes)
-			)
-		)
-		(property "MANUFACTURER" "MPD"
-			(at 210.82 109.22 0)
-			(effects
-				(font
-					(size 1.27 1.27)
-				)
-				(justify bottom)
-				(hide yes)
-			)
-		)
-		(pin "-"
-		)
-		(pin "S1+"
-		)
-		(instances
-			(project ""
-				(path "/6338cb95-8536-41ae-a90a-0bf3cec19d9d/ac09af11-5794-40a5-ab3d-ac2e3f5d0ff8"
-					(reference "BT1")
-					(unit 1)
-				)
